File: PecanPico7.sch (EAGLE design)
At the start: 170 parts, among them IC1 Si4464-B1B-FM, IC10 TC1185-1.8VCT713, IC11 TC1185-2.5VCT713, IC12 ADR380ARTZ, IC13 RF6886, IC14 ALM-GP003, IC15 MPU-9250, IC16 PAC1720-1-AIA-TR, IC2 Si4464-B1B-FM, IC3 BME280_BME280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

Commit message: Tidy up
Connections:
- removed net BOOT1: IC5G$1.PB2
Other:
- note added: "COM"
- note removed: "SDRAM"
Changed lines of the file:
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@@
 <wire x1="190.5" y1="259.08" x2="213.36" y2="259.08" width="0.1524" layer="152"/>
 <wire x1="213.36" y1="259.08" x2="213.36" y2="254" width="0.1524" layer="152"/>
-<text x="132.08" y="255.27" size="2.54" layer="152">SDRAM</text>
-<text x="195.58" y="255.27" size="2.54" layer="152">SDRAM</text>
+<text x="132.08" y="255.27" size="2.54" layer="152">COM</text>
+<text x="195.58" y="255.27" size="2.54" layer="152">COM</text>
 <text x="106.68" y="176.53" size="2.0066" layer="152">SCL
 SDA</text>
@@
 <segment>
 <pinref part="IC5" gate="G$1" pin="PB13"/>
-<wire x1="152.4" y1="167.64" x2="101.6" y2="167.64" width="0.1524" layer="91"/>
-<label x="101.6" y="167.64" size="1.27" layer="95" rot="R180" xref="yes"/>
+<wire x1="152.4" y1="167.64" x2="147.32" y2="167.64" width="0.1524" layer="91"/>
+<label x="147.32" y="167.64" size="1.27" layer="95" rot="R180" xref="yes"/>
 </segment>
 </net>
@@
 <segment>
 <pinref part="IC5" gate="G$1" pin="PB14"/>
-<wire x1="101.6" y1="165.1" x2="152.4" y2="165.1" width="0.1524" layer="91"/>
-<label x="101.6" y="165.1" size="1.27" layer="95" rot="R180" xref="yes"/>
+<wire x1="147.32" y1="165.1" x2="152.4" y2="165.1" width="0.1524" layer="91"/>
+<label x="147.32" y="165.1" size="1.27" layer="95" rot="R180" xref="yes"/>
 </segment>
 </net>
@@
 <segment>
 <pinref part="IC5" gate="G$1" pin="PB15"/>
-<wire x1="152.4" y1="162.56" x2="101.6" y2="162.56" width="0.1524" layer="91"/>
-<label x="101.6" y="162.56" size="1.27" layer="95" rot="R180" xref="yes"/>
+<wire x1="152.4" y1="162.56" x2="147.32" y2="162.56" width="0.1524" layer="91"/>
+<label x="147.32" y="162.56" size="1.27" layer="95" rot="R180" xref="yes"/>
 </segment>
 </net>
@@
 </segment>
 <segment>
-<label x="101.6" y="215.9" size="1.27" layer="95" rot="R180" xref="yes"/>
+<label x="147.32" y="215.9" size="1.27" layer="95" rot="R180" xref="yes"/>
 <pinref part="IC5" gate="G$1" pin="PA11"/>
-<wire x1="152.4" y1="215.9" x2="101.6" y2="215.9" width="0.1524" layer="91"/>
+<wire x1="152.4" y1="215.9" x2="147.32" y2="215.9" width="0.1524" layer="91"/>
 </segment>
 </net>
@@
 <segment>
 <pinref part="IC5" gate="G$1" pin="PB0"/>
-<wire x1="152.4" y1="200.66" x2="101.6" y2="200.66" width="0.1524" layer="91"/>
-<label x="101.6" y="200.66" size="1.27" layer="95" rot="R180" xref="yes"/>
+<wire x1="152.4" y1="200.66" x2="147.32" y2="200.66" width="0.1524" layer="91"/>
+<label x="147.32" y="200.66" size="1.27" layer="95" rot="R180" xref="yes"/>
 </segment>
 </net>
@@
 <segment>
 <pinref part="IC5" gate="G$1" pin="PB11"/>
-<wire x1="101.6" y1="172.72" x2="152.4" y2="172.72" width="0.1524" layer="91"/>
-<label x="101.6" y="172.72" size="1.27" layer="95" rot="R180" xref="yes"/>
+<wire x1="147.32" y1="172.72" x2="152.4" y2="172.72" width="0.1524" layer="91"/>
+<label x="147.32" y="172.72" size="1.27" layer="95" rot="R180" xref="yes"/>
 </segment>
 <segment>
@@
 <segment>
 <pinref part="IC5" gate="G$1" pin="PB10"/>
-<wire x1="152.4" y1="175.26" x2="101.6" y2="175.26" width="0.1524" layer="91"/>
-<label x="101.6" y="175.26" size="1.27" layer="95" rot="R180" xref="yes"/>
+<wire x1="152.4" y1="175.26" x2="147.32" y2="175.26" width="0.1524" layer="91"/>
+<label x="147.32" y="175.26" size="1.27" layer="95" rot="R180" xref="yes"/>
 </segment>
 <segment>
@@
 <segment>
 <pinref part="IC5" gate="G$1" pin="PA14"/>
-<wire x1="101.6" y1="208.28" x2="152.4" y2="208.28" width="0.1524" layer="91"/>
-<label x="101.6" y="208.28" size="1.27" layer="95" rot="R180" xref="yes"/>
+<wire x1="147.32" y1="208.28" x2="152.4" y2="208.28" width="0.1524" layer="91"/>
+<label x="147.32" y="208.28" size="1.27" layer="95" rot="R180" xref="yes"/>
 </segment>
 </net>
@@
 <segment>
 <pinref part="IC5" gate="G$1" pin="PA13"/>
-<wire x1="152.4" y1="210.82" x2="101.6" y2="210.82" width="0.1524" layer="91"/>
-<label x="101.6" y="210.82" size="1.27" layer="95" rot="R180" xref="yes"/>
+<wire x1="152.4" y1="210.82" x2="147.32" y2="210.82" width="0.1524" layer="91"/>
+<label x="147.32" y="210.82" size="1.27" layer="95" rot="R180" xref="yes"/>
 </segment>
 </net>
@@
 <segment>
 <pinref part="IC5" gate="G$1" pin="PB3"/>
-<wire x1="152.4" y1="193.04" x2="101.6" y2="193.04" width="0.1524" layer="91"/>
-<label x="101.6" y="193.04" size="1.27" layer="95" rot="R180" xref="yes"/>
-</segment>
-</net>
-<net name="BOOT1" class="0">
-<segment>
-<pinref part="IC5" gate="G$1" pin="PB2"/>
-<wire x1="152.4" y1="195.58" x2="101.6" y2="195.58" width="0.1524" layer="91"/>
-<label x="101.6" y="195.58" size="1.27" layer="95" rot="R180" xref="yes"/>
+<wire x1="152.4" y1="193.04" x2="147.32" y2="193.04" width="0.1524" layer="91"/>
+<label x="147.32" y="193.04" size="1.27" layer="95" rot="R180" xref="yes"/>
 </segment>
 </net>
@@
 <net name="UART_TO_GPS" class="0">
 <segment>
-<label x="101.6" y="238.76" size="1.27" layer="95" rot="R180" xref="yes"/>
+<label x="147.32" y="238.76" size="1.27" layer="95" rot="R180" xref="yes"/>
 <pinref part="IC5" gate="G$1" pin="PA2"/>
-<wire x1="152.4" y1="238.76" x2="101.6" y2="238.76" width="0.1524" layer="91"/>
+<wire x1="152.4" y1="238.76" x2="147.32" y2="238.76" width="0.1524" layer="91"/>
 </segment>
 <segment>
@@
 <net name="UART_FROM_GPS" class="0">
 <segment>
-<label x="101.6" y="236.22" size="1.27" layer="95" rot="R180" xref="yes"/>
+<label x="147.32" y="236.22" size="1.27" layer="95" rot="R180" xref="yes"/>
 <pinref part="IC5" gate="G$1" pin="PA3"/>
-<wire x1="152.4" y1="236.22" x2="101.6" y2="236.22" width="0.1524" layer="91"/>
+<wire x1="152.4" y1="236.22" x2="147.32" y2="236.22" width="0.1524" layer="91"/>
 </segment>
 <segment>
@@
 <segment>
 <pinref part="IC5" gate="G$2" pin="PE0"/>
-<wire x1="152.4" y1="144.78" x2="101.6" y2="144.78" width="0.1524" layer="91"/>
-<label x="101.6" y="144.78" size="1.27" layer="95" rot="R180" xref="yes"/>
+<wire x1="152.4" y1="144.78" x2="124.46" y2="144.78" width="0.1524" layer="91"/>
+<label x="124.46" y="144.78" size="1.27" layer="95" rot="R180" xref="yes"/>
 </segment>
 </net>
@@
 <segment>
 <pinref part="IC5" gate="G$1" pin="PA15"/>
-<wire x1="152.4" y1="205.74" x2="101.6" y2="205.74" width="0.1524" layer="91"/>
-<label x="101.6" y="205.74" size="1.27" layer="95" rot="R180" xref="yes"/>
+<wire x1="152.4" y1="205.74" x2="147.32" y2="205.74" width="0.1524" layer="91"/>
+<label x="147.32" y="205.74" size="1.27" layer="95" rot="R180" xref="yes"/>
 </segment>
 </net>
@@
 </segment>
 <segment>
-<label x="238.76" y="213.36" size="1.27" layer="95" xref="yes"/>
+<label x="193.04" y="213.36" size="1.27" layer="95" xref="yes"/>
 <pinref part="IC5" gate="G$1" pin="PC12"/>
-<wire x1="238.76" y1="213.36" x2="187.96" y2="213.36" width="0.1524" layer="91"/>
+<wire x1="193.04" y1="213.36" x2="187.96" y2="213.36" width="0.1524" layer="91"/>
 </segment>
 </net>
@@
 <segment>
 <pinref part="IC5" gate="G$1" pin="PC10"/>
-<wire x1="187.96" y1="218.44" x2="238.76" y2="218.44" width="0.1524" layer="91"/>
-<label x="238.76" y="218.44" size="1.27" layer="95" xref="yes"/>
+<wire x1="187.96" y1="218.44" x2="193.04" y2="218.44" width="0.1524" layer="91"/>
+<label x="193.04" y="218.44" size="1.27" layer="95" xref="yes"/>
 </segment>
 </net>
@@
 <segment>
 <pinref part="IC5" gate="G$1" pin="PC11"/>
-<wire x1="187.96" y1="215.9" x2="238.76" y2="215.9" width="0.1524" layer="91"/>
-<label x="238.76" y="215.9" size="1.27" layer="95" xref="yes"/>
+<wire x1="187.96" y1="215.9" x2="193.04" y2="215.9" width="0.1524" layer="91"/>
+<label x="193.04" y="215.9" size="1.27" layer="95" xref="yes"/>
 </segment>
 </net>
@@
 <segment>
 <pinref part="IC5" gate="G$1" pin="PA0"/>
-<wire x1="152.4" y1="243.84" x2="101.6" y2="243.84" width="0.1524" layer="91"/>
-<label x="101.6" y="243.84" size="1.27" layer="95" rot="R180" xref="yes"/>
+<wire x1="152.4" y1="243.84" x2="147.32" y2="243.84" width="0.1524" layer="91"/>
+<label x="147.32" y="243.84" size="1.27" layer="95" rot="R180" xref="yes"/>
 </segment>
 <segment>
@@
 <segment>
 <pinref part="IC5" gate="G$1" pin="PA1"/>
-<wire x1="101.6" y1="241.3" x2="152.4" y2="241.3" width="0.1524" layer="91"/>
-<label x="101.6" y="241.3" size="1.27" layer="95" rot="R180" xref="yes"/>
+<wire x1="147.32" y1="241.3" x2="152.4" y2="241.3" width="0.1524" layer="91"/>
+<label x="147.32" y="241.3" size="1.27" layer="95" rot="R180" xref="yes"/>
 </segment>
 <segment>
@@
 <segment>
 <pinref part="IC5" gate="G$2" pin="PE15"/>
-<wire x1="152.4" y1="106.68" x2="101.6" y2="106.68" width="0.1524" layer="91"/>
-<label x="101.6" y="106.68" size="1.27" layer="95" rot="R180" xref="yes"/>
+<wire x1="152.4" y1="106.68" x2="147.32" y2="106.68" width="0.1524" layer="91"/>
+<label x="147.32" y="106.68" size="1.27" layer="95" rot="R180" xref="yes"/>
 </segment>
 </net>

Commit message: Done many things Replaced 0402 sense resistors by 0603 Fixed LPF at Radio 2 Connected Radio 1 PA to VBAT instead of VCC Corrected MPU9250 GND pad Relocated VBAT signal to avoid interference to MPU9250 Moved parts around
Parts:
- added R43: 0R, sven:RES-04020805
- added SJ2: (no value), PecanPico6:SJ
- R20, R21: value 0.22R -> RES-04020603; device PecanPico6:RES-0402 -> sven:RES-04020603
Connections:
- removed net N$14: C15.2, L6.2, L7.1
- new net N$40: IC4.7_VCC_IO, SJ2.1
- new net N$55: C68.2, C69.2, L11.2, R43.1
- new net N$56: C16.2, L10.1, L7.2
- net N$19: now also C15.2, L6.2, L7.1; no longer C16.2, L10.1, L7.2
- net N$29: now also SJ2.2; no longer IC4.7_VCC_IO
- net VBAT: now also R43.2
- net VCC: no longer C68.2, C69.2, L11.2
Other:
- moved on the sheet: C15, C16, C17, L10, L6, L7
